File: 03_boards/00_bridge_driver/03_kicad/01_main/Drivers.kicad_sch (KiCad schematic)
At the start: 46 parts, among them Q1 SUD90330E, Q2 SUD90330E, Q3 SUD90330E, Q4 SUD90330E, Q5 SUD90330E, Q6 SUD90330E, U1 IRS2104, U2 IRS2104, U3 IRS2104, U4 ISO7740DWR

Commit message: Week 0x8 | Simulation & Objectives (#34)
* Reordered motor folder and rewrote / cleaned up readmes within motors, boards and simulations

* Updated readme logo size

* Made logo 100% width

* Update scaled logo and removed finite element from readme

* Removed objectives

* Removed FEM from readme

* Removed Methodology

* Added a line break before prototype alpha image. Also removed figure naming from the document

* Trying a new formatting technique

* Moved boards link below image

* Removed `REV 2` from image description as its not needed

* Removing overview to see if its good or not

* Trying a new formatting style

* Removed the top line section

* Removed prototype from naming schema

* Changed top block

* Updated shields and updated description

* Removed some pose & added alpha and beta symbols because their cool

* Added a line break below documentation

* Added objectives to readme

* Removed the indexing from two notes

* Renamed `motor notes` with `alpha notes`

* Indexed the conceptual and removed : from note

* Updated parameter files and added short note about analytical model

* Cleaned up analytical model

* Updated analytical simulation

* Updated readmes for analytical model

* Updated the electrical equations

* Updated formatting for motors & boards

* Updated readmes and added sections to openLSM main readme

* I like it as a code block more

* Objectives should be in overview

* Moved aspirations note below objectives

* Made it more broad to contents than designs and contributions

* Updated subsection heading?

* Removed the "accurate dynamics" note its bad filler

* Removed TBD from readme

* Reformatting the tags section in documentation

* Updated analytical model

* Final iteration of analytical model before documentation

* Removing the global warning should be upto the individual readmes to say so

* Renamed metric.ut to derived.ut

* Added flow diagram for analytical model

* Updated the readmes to reflect uncertainty in the actual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
Connections:
- net at Q5.2 (G), R8.2: now also D7.2 (A); no longer D7.1 (K)
- net at R3.2, U1.5 (LO): now also D3.1 (K); no longer D3.2 (A)
- net at R2.1, U1.7 (HO): now also D2.1 (K); no longer D2.2 (A)
- net at Q1.2 (G), R2.2: now also D2.2 (A); no longer D2.1 (K)
- net at R5.1, U2.7 (HO): now also D12.1 (K); no longer D12.2 (A)
- net at Q3.2 (G), R5.2: now also D12.2 (A); no longer D12.1 (K)
- net at Q6.2 (G), R9.1: now also D8.2 (A); no longer D8.1 (K)
- net at R9.2, U3.5 (LO): now also D8.1 (K); no longer D8.2 (A)
- net at R6.2, U2.5 (LO): now also D13.1 (K); no longer D13.2 (A)
- net at Q2.2 (G), R3.1: now also D3.2 (A); no longer D3.1 (K)
- net at R8.1, U3.7 (HO): now also D7.1 (K); no longer D7.2 (A)
- net at Q4.2 (G), R6.1: now also D13.2 (A); no longer D13.1 (K)
Other:
- note added: "F, C"
- moved on the sheet: C10, C11, D12, D2, D7, R10, U4

Commit message: More footprint selection. YAY
Parts:
- removed Q1, Q2, Q3, Q4, Q5, Q6: SUD90330E, symbol Simulation_SPICE:NMOS
- added Q1, Q2, Q3, Q4, Q5, Q6: SUD90330E, sud90330e:TO-252-2, symbol Transistor_FET:Q_NMOS_GSD
- R1, R10, R2, R3, R4, R5, R6, R7, R8, R9: footprint (none) -> Resistor_SMD:R_0603_1608Metric
- U1, U2, U3: footprint (none) -> Package_SO:SOIC-8_3.9x4.9mm_P1.27mm
Connections:
- net PA_CS: now also Q1.2 (S), Q2.3 (D)
- net PB_CS: now also Q5.2 (S), Q6.3 (D)
- net PC_CS: now also Q3.2 (S), Q4.3 (D)
- net PGND: now also Q2.2 (S), Q4.2 (S), Q6.2 (S)
- net PVCC: now also Q1.3 (D), Q3.3 (D), Q5.3 (D)
- net at D7.2 (A), R8.2: now also Q3.1 (G)
- net at D2.2 (A), R2.2: now also Q1.1 (G)
- net at D12.2 (A), R5.2: now also Q5.1 (G)
- net at D8.2 (A), R9.1: now also Q4.1 (G)
- net at D3.2 (A), R3.1: now also Q2.1 (G)
- net at D13.2 (A), R6.1: now also Q6.1 (G)
Other:
- note removed: "F, C"

Commit message: Footprints finished and hence initial BOM based on footprints is also
Parts:
- C1, C10, C11, C4, C7: footprint (none) -> Capacitor_SMD:C_0603_1608Metric
- C2, C6, C9: footprint (none) -> Capacitor_SMD:C_1206_3216Metric
- C3, C5, C8: value 100uF -> 220uF; footprint (none) -> Capacitor_THT:CP_Radial_D8.0mm_P3.50mm
- D1, D10, D11, D12, D13, D14, D15, D2, D3, D4, D5, D6, D7, D8, D9: footprint (none) -> ES1D:DIOM4325X250N
Changed lines of the file:
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@@
 			)
 		)
-		(property "Footprint" ""
+		(property "Footprint" "ES1D:DIOM4325X250N"
 			(at 120.65 111.76 0)
 			(hide yes)
@@
 			)
 		)
-		(property "Footprint" ""
+		(property "Footprint" "Capacitor_SMD:C_0603_1608Metric"
 			(at 145.7452 49.53 0)
 			(hide yes)
@@
 			)
 		)
-		(property "Footprint" ""
+		(property "Footprint" "Capacitor_SMD:C_0603_1608Metric"
 			(at 240.9952 106.68 0)
 			(hide yes)
@@
 			)
 		)
-		(property "Footprint" ""
+		(property "Footprint" "ES1D:DIOM4325X250N"
 			(at 120.65 41.91 0)
 			(hide yes)
@@
 			)
 		)
-		(property "Footprint" ""
+		(property "Footprint" "ES1D:DIOM4325X250N"
 			(at 207.01 63.5 0)
 			(hide yes)
@@
 			)
 		)
-		(property "Footprint" ""
+		(property "Footprint" "Capacitor_SMD:C_0603_1608Metric"
 			(at 26.3652 50.8 0)
 			(hide yes)
@@
 			)
 		)
-		(property "Footprint" ""
+		(property "Footprint" "ES1D:DIOM4325X250N"
 			(at 74.93 27.94 0)
 			(hide yes)
@@
 			)
 		)
-		(property "Footprint" ""
+		(property "Footprint" "Capacitor_SMD:C_1206_3216Metric"
 			(at 199.0852 49.53 0)
 			(hide yes)
@@
 			)
 		)
-		(property "Footprint" ""
+		(property "Footprint" "ES1D:DIOM4325X250N"
 			(at 194.31 26.67 0)
 			(hide yes)
@@
 			)
 		)
-		(property "Footprint" ""
+		(property "Footprint" "ES1D:DIOM4325X250N"
 			(at 120.65 99.06 0)
 			(hide yes)
@@
 			)
 		)
-		(property "Footprint" ""
+		(property "Footprint" "Capacitor_SMD:C_1206_3216Metric"
 			(at 79.7052 50.8 0)
 			(hide yes)
@@
 			)
 		)
-		(property "Footprint" ""
+		(property "Footprint" "ES1D:DIOM4325X250N"
 			(at 87.63 88.9 0)
 			(hide yes)
@@
 			)
 		)
-		(property "Footprint" ""
+		(property "Footprint" "ES1D:DIOM4325X250N"
 			(at 120.65 53.34 0)
 			(hide yes)
@@
 			)
 		)
-		(property "Footprint" ""
+		(property "Footprint" "Capacitor_SMD:C_1206_3216Metric"
 			(at 79.7052 107.95 0)
 			(hide yes)
@@
 			)
 		)
-		(property "Footprint" ""
+		(property "Footprint" "ES1D:DIOM4325X250N"
 			(at 87.63 31.75 0)
 			(hide yes)
@@
 			)
 		)
-		(property "Footprint" ""
+		(property "Footprint" "ES1D:DIOM4325X250N"
 			(at 87.63 121.92 0)
 			(hide yes)
@@
 			)
 		)
-		(property "Value" "100uF"
+		(property "Value" "220uF"
 			(at 39.37 47.3709 0)
 			(show_name no)
@@
 			)
 		)
-		(property "Footprint" ""
+		(property "Footprint" "Capacitor_THT:CP_Radial_D8.0mm_P3.50mm"
 			(at 36.5252 50.8 0)
 			(hide yes)
@@
 			)
 		)
-		(property "Value" "100uF"
+		(property "Value" "220uF"
 			(at 158.75 46.1009 0)
 			(show_name no)
@@
 			)
 		)
-		(property "Footprint" ""
+		(property "Footprint" "Capacitor_THT:CP_Radial_D8.0mm_P3.50mm"
 			(at 155.9052 49.53 0)
 			(hide yes)
@@
 			)
 		)
-		(property "Value" "100uF"
+		(property "Value" "220uF"
 			(at 39.37 104.5209 0)
 			(show_name no)
@@
 			)
 		)
-		(property "Footprint" ""
+		(property "Footprint" "Capacitor_THT:CP_Radial_D8.0mm_P3.50mm"
 			(at 36.5252 107.95 0)
 			(hide yes)
@@
 			)
 		)
-		(property "Footprint" ""
+		(property "Footprint" "ES1D:DIOM4325X250N"
 			(at 240.03 53.34 0)
 			(hide yes)
@@
 			)
 		)
-		(property "Footprint" ""
+		(property "Footprint" "ES1D:DIOM4325X250N"
 			(at 240.03 40.64 0)
 			(hide yes)
@@
 			)
 		)
-		(property "Footprint" ""
+		(property "Footprint" "Capacitor_SMD:C_0603_1608Metric"
 			(at 228.2952 106.68 0)
 			(hide yes)
@@
 			)
 		)
-		(property "Footprint" ""
+		(property "Footprint" "ES1D:DIOM4325X250N"
 			(at 207.01 30.48 0)
 			(hide yes)
@@
 			)
 		)
-		(property "Footprint" ""
+		(property "Footprint" "ES1D:DIOM4325X250N"
 			(at 87.63 64.77 0)
 			(hide yes)
@@
 			)
 		)
-		(property "Footprint" ""
+		(property "Footprint" "Capacitor_SMD:C_0603_1608Metric"
 			(at 26.3652 107.95 0)
 			(hide yes)
@@
 			)
 		)
-		(property "Footprint" ""
+		(property "Footprint" "ES1D:DIOM4325X250N"
 			(at 74.93 85.09 0)
 			(hide yes)

Commit message: Added work so far on bridge driver. Took some pics and updates readmes.
Parts:
- removed D12, D13, D2, D3, D7, D8: ES1D, ES1D:DIOM4325X250N, symbol Device:D
- R2, R3, R5, R6, R8, R9: footprint Resistor_SMD:R_0603_1608Metric -> Resistor_SMD:R_1206_3216Metric
