File: 03_boards/00_bridge_driver/03_kicad/01_main/main.kicad_pcb (KiCad board)
At the start: 2 copper layers, 9 parts, among them U10 INA241A3xD, U11 INA241A3xD, U5 STM32G431K8Tx, U6 MAX3485, U7 LD1117V33, U8 LM2596S-5, U9 LM2596S-12

Commit message: More footprint selection. YAY
Parts:
- added FB1: BLM18AG601SN1D, BLM18AG601SN1D:BEADC1608X95N, F.Cu at (88.4, 129.9)
- added L5: 82103C, 82103C:IND_8200_MUR, F.Cu at (90.2, 126.2)
- added STEP1: 01x02, Connector_JST:JST_PH_B2B-PH-K_1x02_P2.00mm_Vertical, F.Cu at (89.4, 119.9)
- added SW1: SW_Push, Button_Switch_SMD:SW_Push_1P1T_NO_CK_KMR2, F.Cu at (90.7, 135.3)
- added SW2: SW_Push, Button_Switch_SMD:SW_Push_1P1T_NO_CK_KMR2, F.Cu at (90.7, 140.0)
- added U1: IRS2104, Package_SO:SOIC-8_3.9x4.9mm_P1.27mm, F.Cu at (100.6, 140.2)
- added U10: REF3020, Package_TO_SOT_SMD:SOT-23, F.Cu at (112.5, 132.6)
- added U11: INA241A2xD, Package_SO:SOIC-8_3.9x4.9mm_P1.27mm, F.Cu at (114.3, 120.6)
- added U12: AMC1311, AMC1311DWVR:DWV0008A, F.Cu at (103.2, 120.7)
- added U13: AMC1311, AMC1311DWVR:DWV0008A, F.Cu at (103.2, 127.8)
- added U14: CME0512S3C, CME0512S3C:CME_SC_MUR, F.Cu at (76.0, 123.2)
- added U15: CME0303S3C, CME0512S3C:CME_SC_MUR, F.Cu at (76.0, 131.1)
- added U16: INA241A2xD, Package_SO:SOIC-8_3.9x4.9mm_P1.27mm, F.Cu at (114.3, 127.1)
- added U2: IRS2104, Package_SO:SOIC-8_3.9x4.9mm_P1.27mm, F.Cu at (100.6, 146.8)
- added U3: IRS2104, Package_SO:SOIC-8_3.9x4.9mm_P1.27mm, F.Cu at (100.6, 153.3)
- added U4: ISO7740DWR, ISO7740DWR:SOIC127P1030X265-16N, F.Cu at (111.8, 142.7)
- added Y1: ECS-80-20-18-TR, ECS-80-18-23B-JTN-TR:XTAL_ECS-80-20-18-TR, F.Cu at (80.7, 136.8)

Commit message: More footprints.
Parts:
- added CAN1: 01x02, Connector_JST:JST_PH_B2B-PH-K_1x02_P2.00mm_Vertical, F.Cu at (57.5, 127.7)
- added D16: LED, LED_SMD:LED_0603_1608Metric_Pad1.05x0.95mm_HandSolder, F.Cu at (52.7, 139.8)
- added INT1: 01x04, Connector_JST:JST_PH_B4B-PH-K_1x04_P2.00mm_Vertical, F.Cu at (57.5, 114.6)
- added J1: 01x02, Connector_Wire:SolderWire-1sqmm_1x02_P7.8mm_D1.4mm_OD3.9mm_Relief, F.Cu at (39.5, 114.8)
- added PH1: 01x03, Connector_Wire:SolderWire-2.5sqmm_1x03_P7.2mm_D2.4mm_OD3.6mm_Relief, F.Cu at (16.0, 130.2)
- added PRO1: 01x06, Connector_JST:JST_PH_B6B-PH-K_1x06_P2.00mm_Vertical, F.Cu at (53.5, 134.7)
- added Q1: SUD90330E, sud90330e:TO-252-2, F.Cu at (20.2, 79.5)
- added Q2: SUD90330E, sud90330e:TO-252-2, F.Cu at (20.2, 87.6)
- added Q3: SUD90330E, sud90330e:TO-252-2, F.Cu at (20.2, 95.6)
- added Q4: SUD90330E, sud90330e:TO-252-2, F.Cu at (20.2, 103.7)
- added Q5: SUD90330E, sud90330e:TO-252-2, F.Cu at (20.2, 111.7)
- added Q6: SUD90330E, sud90330e:TO-252-2, F.Cu at (20.2, 119.8)
- added R1: 5, Resistor_SMD:R_0603_1608Metric, F.Cu at (28.3, 76.8)
- added R10: 4.7k, Resistor_SMD:R_0603_1608Metric, F.Cu at (32.3, 86.8)
- added R11: 120, Resistor_SMD:R_0603_1608Metric, F.Cu at (52.5, 113.1)
- added R12: 10, Resistor_SMD:R_0603_1608Metric, F.Cu at (52.5, 115.6)
- added R13: 10, Resistor_SMD:R_0603_1608Metric, F.Cu at (52.5, 118.1)
- added R14: 220, Resistor_SMD:R_0603_1608Metric, F.Cu at (52.5, 120.7)
- added R15: 220, Resistor_SMD:R_0603_1608Metric, F.Cu at (52.5, 123.2)
- added R16: 10K, Resistor_SMD:R_0603_1608Metric, F.Cu at (52.5, 125.7)
- added R17: 10K, Resistor_SMD:R_0603_1608Metric, F.Cu at (52.5, 128.2)
- added R18: 220, Resistor_SMD:R_0603_1608Metric, F.Cu at (52.5, 130.7)
- added R19: 10mOhm, Resistor_SMD:R_2512_6332Metric, F.Cu at (40.6, 78.0)
- added R2: 47, Resistor_SMD:R_0603_1608Metric, F.Cu at (28.3, 79.3)
- added R20: 10mOhm, Resistor_SMD:R_2512_6332Metric, F.Cu at (40.6, 82.9)
- added R21: 10mOhm, Resistor_SMD:R_2512_6332Metric, F.Cu at (40.6, 87.8)
- added R22: 0 Ohm, Resistor_SMD:R_2512_6332Metric, F.Cu at (40.6, 92.7)
- added R23: 0 Ohm, Resistor_SMD:R_2512_6332Metric, F.Cu at (40.6, 97.6)
- added R24: 0 Ohm, Resistor_SMD:R_2512_6332Metric, F.Cu at (40.6, 102.5)
- added R25: 3mOhm, Resistor_SMD:R_2512_6332Metric, F.Cu at (40.6, 107.4)
- added R26: 3mOhm, Resistor_SMD:R_2512_6332Metric, F.Cu at (49.3, 78.0)
- added R27: 3mOhm, Resistor_SMD:R_2512_6332Metric, F.Cu at (49.3, 82.9)
- added R28: 0 Ohm, Resistor_SMD:R_2512_6332Metric, F.Cu at (49.3, 87.8)
- added R29: 0 Ohm, Resistor_SMD:R_2512_6332Metric, F.Cu at (49.3, 92.7)
- added R3: 47, Resistor_SMD:R_0603_1608Metric, F.Cu at (28.3, 81.8)
- added R30: 0 Ohm, Resistor_SMD:R_2512_6332Metric, F.Cu at (49.3, 97.6)
- added R31: 1mOhm, Resistor_SMD:R_2512_6332Metric, F.Cu at (49.3, 102.5)
- added R32: 1mOhm, Resistor_SMD:R_2512_6332Metric, F.Cu at (49.3, 107.4)
- added R33: 1mOhm, Resistor_SMD:R_2512_6332Metric, F.Cu at (58.0, 78.0)
- added R34: 0 Ohm, Resistor_SMD:R_2512_6332Metric, F.Cu at (58.0, 82.9)
- added R35: 0 Ohm, Resistor_SMD:R_2512_6332Metric, F.Cu at (58.0, 87.8)
- added R36: 0 Ohm, Resistor_SMD:R_2512_6332Metric, F.Cu at (58.0, 92.7)
- added R4: 5, Resistor_SMD:R_0603_1608Metric, F.Cu at (28.3, 84.3)
- added R5: 47, Resistor_SMD:R_0603_1608Metric, F.Cu at (28.3, 86.8)
- added R6: 47, Resistor_SMD:R_0603_1608Metric, F.Cu at (32.3, 76.8)
- added R7: 5, Resistor_SMD:R_0603_1608Metric, F.Cu at (32.3, 79.3)
- added R8: 47, Resistor_SMD:R_0603_1608Metric, F.Cu at (32.3, 81.8)
- added R9: 47, Resistor_SMD:R_0603_1608Metric, F.Cu at (32.3, 84.3)
- D17, D18: footprint Diode_THT:D_DO-201AD_P15.24mm_Horizontal -> Diode_SMD:D_SMC
- U7: footprint Package_TO_SOT_THT:TO-220-3_Vertical -> Package_TO_SOT_SMD:SOT-223
- renumbered L5 to L4

Commit message: Footprints finished and hence initial BOM based on footprints is also
Parts:
- added C1: 1uF, Capacitor_SMD:C_0603_1608Metric, F.Cu at (58.8, 170.5)
- added C10: 1uF, Capacitor_SMD:C_0603_1608Metric, F.Cu at (58.8, 178.0)
- added C11: 1uF, Capacitor_SMD:C_0603_1608Metric, F.Cu at (58.8, 180.5)
- added C12: 30pf, Capacitor_SMD:C_0603_1608Metric, F.Cu at (81.1, 150.0)
- added C13: 30pf, Capacitor_SMD:C_0603_1608Metric, F.Cu at (81.1, 152.5)
- added C14: 100nf, Capacitor_SMD:C_0603_1608Metric, F.Cu at (81.1, 155.0)
- added C15: 100nf, Capacitor_SMD:C_0603_1608Metric, F.Cu at (81.1, 157.5)
- added C16: 10uf, Capacitor_SMD:C_0603_1608Metric, F.Cu at (81.1, 160.0)
- added C17: 100nf, Capacitor_SMD:C_0603_1608Metric, F.Cu at (81.1, 162.5)
- added C18: 1uf, Capacitor_SMD:C_0603_1608Metric, F.Cu at (81.1, 165.0)
- added C19: 10uf, Capacitor_SMD:C_1206_3216Metric, F.Cu at (85.9, 150.4)
- added C2: 10uF, Capacitor_SMD:C_1206_3216Metric, F.Cu at (53.9, 170.9)
- added C20: 22uf, Capacitor_SMD:C_1206_3216Metric, F.Cu at (85.9, 153.7)
- added C21: 100nf, Capacitor_SMD:C_0603_1608Metric, F.Cu at (81.1, 167.5)
- added C26: 0.68uF, Capacitor_SMD:C_1206_3216Metric, F.Cu at (85.9, 157.1)
- added C27: 4.7uF, Capacitor_SMD:C_1206_3216Metric, F.Cu at (85.9, 160.4)
- added C28: 10uF, Capacitor_SMD:C_1206_3216Metric, F.Cu at (81.9, 172.5)
- added C4: 1uF, Capacitor_SMD:C_0603_1608Metric, F.Cu at (58.8, 173.0)
- added C6: 10uF, Capacitor_SMD:C_1206_3216Metric, F.Cu at (53.9, 174.3)
- added C7: 1uF, Capacitor_SMD:C_0603_1608Metric, F.Cu at (58.8, 175.5)
- added C9: 10uF, Capacitor_SMD:C_1206_3216Metric, F.Cu at (53.9, 177.6)
- added D1: ES1D, ES1D:DIOM4325X250N, F.Cu at (55.8, 150.8)
- added D10: ES1D, ES1D:DIOM4325X250N, F.Cu at (64.5, 167.2)
- added D11: ES1D, ES1D:DIOM4325X250N, F.Cu at (73.1, 150.8)
- added D12: ES1D, ES1D:DIOM4325X250N, F.Cu at (73.1, 154.9)
- added D13: ES1D, ES1D:DIOM4325X250N, F.Cu at (73.1, 159.0)
- added D14: ES1D, ES1D:DIOM4325X250N, F.Cu at (73.1, 163.1)
- added D15: ES1D, ES1D:DIOM4325X250N, F.Cu at (73.1, 167.2)
- added D2: ES1D, ES1D:DIOM4325X250N, F.Cu at (55.8, 154.9)
- added D3: ES1D, ES1D:DIOM4325X250N, F.Cu at (55.8, 159.0)
- added D4: ES1D, ES1D:DIOM4325X250N, F.Cu at (55.8, 163.1)
- added D5: ES1D, ES1D:DIOM4325X250N, F.Cu at (55.8, 167.2)
- added D6: ES1D, ES1D:DIOM4325X250N, F.Cu at (64.5, 150.8)
- added D7: ES1D, ES1D:DIOM4325X250N, F.Cu at (64.5, 154.9)
- added D8: ES1D, ES1D:DIOM4325X250N, F.Cu at (64.5, 159.0)
- added D9: ES1D, ES1D:DIOM4325X250N, F.Cu at (64.5, 163.1)
- added L3: 82683C, 82683C:FUSE_MF-USMFLAB, F.Cu at (85.8, 164.2)
- J1: footprint Connector_Wire:SolderWire-1sqmm_1x02_P7.8mm_D1.4mm_OD3.9mm_Relief -> Connector_Wire:SolderWire-1sqmm_1x02_P7.8mm_D1.4mm_OD3.9mm

Commit message: Initial PCB modelling work
Parts:
- removed R22, R23, R24, R28, R29, R30, R34, R35, R36: 0 Ohm, Resistor_SMD:R_2512_6332Metric
- removed R25, R26, R27: 3mOhm, Resistor_SMD:R_2512_6332Metric
- removed R31, R32, R33: 1mOhm, Resistor_SMD:R_2512_6332Metric
- removed the U10 at (117.6, 79.1)
- removed the U10 at (112.5, 132.6)
- removed the U11 at (114.3, 120.6)
- removed the U11 at (117.6, 85.6)
- added C22: 680uF, Capacitor_THT:CP_Radial_D10.0mm_P5.00mm, F.Cu at (-87.6, 20.5)
- added C23: 220uF, Capacitor_THT:CP_Radial_D8.0mm_P3.50mm, F.Cu at (-81.7, -5.22)
- added C24: 680uF, Capacitor_THT:CP_Radial_D10.0mm_P5.00mm, F.Cu at (-87.6, 32.0)
- added C25: 220uF, Capacitor_THT:CP_Radial_D8.0mm_P3.50mm, F.Cu at (-81.7, 4.33)
- added C3: 220uF, Capacitor_THT:CP_Radial_D8.0mm_P3.50mm, F.Cu at (-49.4, 15.3)
- added C5: 220uF, Capacitor_THT:CP_Radial_D8.0mm_P3.50mm, F.Cu at (-49.4, 24.9)
- added C8: 220uF, Capacitor_THT:CP_Radial_D8.0mm_P3.50mm, F.Cu at (-49.4, 34.4)
- added J2: Conn_01x01, Connector_Wire:SolderWire-2.5sqmm_1x01_D2.4mm_OD3.6mm, F.Cu at (40.0, 6.00)
- added J3: Conn_01x01, Connector_Wire:SolderWire-2.5sqmm_1x01_D2.4mm_OD3.6mm, F.Cu at (40.0, 54.0)
- added L1: 33uH, Inductor_SMD:L_Bourns_SRR1260, F.Cu at (-111.6, 21.7)
- added L2: 68uH, Inductor_SMD:L_Bourns_SRR1260, F.Cu at (-111.6, 35.8)
- added U10: REF3020, Package_TO_SOT_SMD:SOT-23, F.Cu at (-62.3, 61.5)
- added U11: INA241A2xD, Package_SO:SOIC-8_3.9x4.9mm_P1.27mm, B.Cu at (53.4, 15.1)
- J1: footprint Connector_Wire:SolderWire-1sqmm_1x02_P7.8mm_D1.4mm_OD3.9mm -> Connector_Wire:SolderWire-0.5sqmm_1x02_P4.6mm_D0.9mm_OD2.1mm
- R19, R20, R21: value 10mOhm -> 5mOhm; moved to B.Cu
- U16: moved to B.Cu
- moved U9 302.2 mm to (-137.4, 3.20)
- moved U8 272.5 mm to (-107.9, -3.83)
- moved U6 264.8 mm to (-71.0, -6.64)
- moved U5 257.4 mm to (-85.5, 43.5)
- moved C18 223.6 mm to (-98.5, 31.8)
- moved C21 223.6 mm to (-98.5, 34.3)
- moved Y1 221.0 mm to (-93.2, 0.38)
- moved C12 218.4 mm to (-102.5, 31.8)
- moved C13 218.4 mm to (-102.5, 34.3)
- moved C14 218.4 mm to (-102.5, 36.8)
- moved C15 218.4 mm to (-102.5, 39.3)
- moved C16 218.4 mm to (-102.5, 41.8)
- moved C17 218.4 mm to (-102.5, 44.3)
- moved PRO1 207.6 mm to (-97.9, -7.28)
- moved FB1 207.5 mm to (-82.9, 12.9)
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Connections:
- PH1 pad 1: PC -> C_IN-
- PH1 pad 3: PA -> A_IN-
- Q3 pad 2: PC_CS -> C_IN+
- Q4 pad 3: PC_CS -> C_IN+
- Q5 pad 2: B_IN+ -> PB_CS
- Q6 pad 3: B_IN+ -> PB_CS
- R19 pad 1: B_IN+ -> PB_CS
- R19 pad 2: B_IN- -> PB
- R21 pad 1: PC_CS -> C_IN+
- R21 pad 2: Net-(R21-Pad2) -> C_IN-
- U16 pad 1: B_IN- -> C_IN-
- U16 pad 8: B_IN+ -> C_IN+
Routing:
- net PVCC: track 0.00 -> 53.3 mm
- net PGND: track 0.00 -> 48.8 mm
- net A_IN-: track 0.00 -> 18.0 mm
- net C_IN-: track 0.00 -> 14.7 mm
- net A_IN+: track 0.00 -> 11.9 mm
- net C_IN+: track 0.00 -> 8.32 mm
- net PB: track 0.00 -> 6.08 mm
- net (no net): vias 0 -> 4
Other:
- board outline added: 80 x 60 mm

Commit message: Added work so far on bridge driver. Took some pics and updates readmes.
Parts:
- removed D12, D13, D2, D3, D7, D8: ES1D, ES1D:DIOM4325X250N
- PH1: footprint Connector_Wire:SolderWire-2.5sqmm_1x03_P7.2mm_D2.4mm_OD3.6mm_Relief -> Connector_Wire:SolderWire-2.5sqmm_1x03_P7.2mm_D2.4mm_OD3.6mm
- R2, R3, R5, R6, R8, R9: footprint Resistor_SMD:R_0603_1608Metric -> Resistor_SMD:R_1206_3216Metric
- U12, U13, U4: moved to B.Cu
- moved U14 131.6 mm to (25.2, 56.0)
- moved U15 128.5 mm to (25.2, 7.50)
- moved INT1 121.1 mm to (19.3, 55.2), turned to 180 degrees
- moved PRO1 116.3 mm to (5.50, 46.0), turned to 90 degrees
- moved VCC1 111.3 mm to (13.9, 7.40)
- moved U5 102.6 mm to (17.1, 39.9)
- moved U13 86.4 mm to (29.0, 15.0), turned to 180 degrees
- moved STEP1 80.6 mm to (5.50, 27.3), turned to 90 degrees
- moved CAN1 79.7 mm to (5.50, 17.0), turned to 90 degrees
- moved U12 78.2 mm to (29.0, 45.0), turned to 180 degrees
- moved U3 75.8 mm to (35.0, 45.0)
- moved U2 74.3 mm to (35.0, 30.0)
- moved U1 73.7 mm to (35.0, 15.0)
- moved R9 72.7 mm to (39.0, 50.0), turned to 180 degrees
- moved C9 72.7 mm to (36.0, 39.7), turned to 180 degrees
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- renumbered J3 to PGND1, J2 to PVCC1, J1 to VCC1
Routing:
- net PB_CS: track 0.00 -> 27.0 mm, vias 0 -> 1
- net A_IN-: track 18.0 -> 6.14 mm
- net C_IN-: track 14.7 -> 5.94 mm
- net Net-(U2-VS): track 0.00 -> 7.83 mm
- net Net-(U3-VS): track 0.00 -> 7.71 mm
- net Net-(U1-VS): track 0.00 -> 7.22 mm
- net PVCC: track 53.3 -> 46.7 mm
- net C_IN+: track 8.32 -> 14.5 mm, vias 0 -> 1
- net PGND: track 48.8 -> 53.2 mm
- net Net-(U3-HO): track 0.00 -> 4.03 mm
- net Net-(U1-HO): track 0.00 -> 4.03 mm
- net Net-(U2-HO): track 0.00 -> 4.03 mm
- net A_IN+: track 11.9 -> 15.8 mm, vias 0 -> 1
- net Net-(D1-K): track 0.00 -> 3.94 mm
- net Net-(D6-K): track 0.00 -> 3.49 mm
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- added copper zone on B.Cu, net PGND
Other:
- copper layers 2 -> 4
- board text added: "PA"
- board text added: "PB"
- board text added: "PC"
