File: 03_boards/00_bridge_driver/03_kicad/01_main/main.kicad_pcb (KiCad board)
At the start: 2 copper layers, 9 parts, among them U10 INA241A3xD, U11 INA241A3xD, U5 STM32G431K8Tx, U6 MAX3485, U7 LD1117V33, U8 LM2596S-5, U9 LM2596S-12

Commit message: Week 0x9 | Nearly there! (#38)
* Updated readmes formatting & other files

* Removed no commercial aspiration notes and added a simple status section for the readme

* Made the status section inline

* Forgot a full stop.

* Added application notes to docs/readme.md

* Added current state and terminal state on the application notes series

* Added .md instead of .csv for BOM

* Added BOM for bridge driver and updated the - to em

* Added 04_procurement folders and made 04_media into 05_media

* Added fixture folder and moved docs to 00

* Technically I have done that just by the bridge driver design.

* Added checking system for BOM and added 05_media section for bridge driver

* Added the order for magnetic encoder

* Added the the link to the digikey file.

* Updated media & readmes to reflect that

* Got the digikey BOM and also checked the list off for armature board

* Nearly finished the schematic for driver board

* Added a some code and fixed the derived.ut vs metric.ut referencing mistake

* Finished Driver Board Schematic.

* More footprint selection. YAY

* More footprints.

* Footprints finished and hence initial BOM based on footprints is also

* Updated schematic.

* Improving the unit boundary and notes for 00_analytical

* Updated main readme to reflect work done this week.

* Removed the line about the integrated sensor board. it's literally below it.

* Rewrote fabrication note.

* Update README.md

* Updated readmes and added the bowley system logo

* Made it clear the values and updated the schematics.

* Updated comment to design not development. they mean different things.

* deleted .csv -> Who uses it anyways!?

* Initial PCB modelling work

* Added work so far on bridge driver. Took some pics and updates readmes.

* Updated to doubles images (back and front)
Parts:
- added C1: 1uF, Capacitor_SMD:C_0603_1608Metric, F.Cu at (-32.4, 11.8)
- added C10: 1uF, Capacitor_SMD:C_0603_1608Metric, F.Cu at (-32.4, 19.3)
- added C11: 1uF, Capacitor_SMD:C_0603_1608Metric, F.Cu at (-32.4, 21.8)
- added C12: 30pf, Capacitor_SMD:C_0603_1608Metric, F.Cu at (-102.5, 31.8)
- added C13: 30pf, Capacitor_SMD:C_0603_1608Metric, F.Cu at (-102.5, 34.3)
- added C14: 100nf, Capacitor_SMD:C_0603_1608Metric, F.Cu at (-102.5, 36.8)
- added C15: 100nf, Capacitor_SMD:C_0603_1608Metric, F.Cu at (-102.5, 39.3)
- added C16: 10uf, Capacitor_SMD:C_0603_1608Metric, F.Cu at (-102.5, 41.8)
- added C17: 100nf, Capacitor_SMD:C_0603_1608Metric, F.Cu at (-102.5, 44.3)
- added C18: 1uf, Capacitor_SMD:C_0603_1608Metric, F.Cu at (-98.5, 31.8)
- added C19: 10uf, Capacitor_SMD:C_1206_3216Metric, F.Cu at (-49.1, 32.8)
- added C2: 10uF, Capacitor_SMD:C_1206_3216Metric, F.Cu at (37.8, 9.20)
- added C20: 22uf, Capacitor_SMD:C_1206_3216Metric, F.Cu at (-51.0, 41.5)
- added C21: 100nf, Capacitor_SMD:C_0603_1608Metric, F.Cu at (-98.5, 34.3)
- added C22: 680uF, Capacitor_THT:CP_Radial_D10.0mm_P5.00mm, F.Cu at (-21.2, 32.7)
- added C23: 220uF, Capacitor_THT:CP_Radial_D8.0mm_P3.50mm, F.Cu at (-81.7, -5.22)
- added C24: 680uF, Capacitor_THT:CP_Radial_D10.0mm_P5.00mm, F.Cu at (-36.1, 39.5)
- added C25: 220uF, Capacitor_THT:CP_Radial_D8.0mm_P3.50mm, F.Cu at (-81.7, 4.33)
- added C26: 0.68uF, Capacitor_SMD:C_1206_3216Metric, F.Cu at (-69.9, 46.9)
- added C27: 4.7uF, Capacitor_SMD:C_1206_3216Metric, F.Cu at (-69.9, 50.2)
- added C28: 10uF, Capacitor_SMD:C_1206_3216Metric, F.Cu at (-18.0, 59.8)
- added C3: 220uF, Capacitor_THT:CP_Radial_D8.0mm_P3.50mm, F.Cu at (-49.4, 15.3)
- added C4: 1uF, Capacitor_SMD:C_0603_1608Metric, F.Cu at (-32.4, 14.3)
- added C5: 220uF, Capacitor_THT:CP_Radial_D8.0mm_P3.50mm, F.Cu at (-13.9, 23.0)
- added C6: 10uF, Capacitor_SMD:C_1206_3216Metric, F.Cu at (36.0, 24.6)
- added C7: 1uF, Capacitor_SMD:C_0603_1608Metric, F.Cu at (-32.4, 16.8)
- added C8: 220uF, Capacitor_THT:CP_Radial_D8.0mm_P3.50mm, F.Cu at (-24.0, 18.0)
- added C9: 10uF, Capacitor_SMD:C_1206_3216Metric, F.Cu at (36.0, 39.7)
- added CAN1: 01x02, Connector_JST:JST_PH_B2B-PH-K_1x02_P2.00mm_Vertical, F.Cu at (5.50, 17.0)
- added D1: ES1D, ES1D:DIOM4325X250N, F.Cu at (-50.8, -53.1)
- added D10: ES1D, ES1D:DIOM4325X250N, F.Cu at (-50.8, -32.6)
- added D11: ES1D, ES1D:DIOM4325X250N, F.Cu at (-50.8, -28.4)
- added D14: ES1D, ES1D:DIOM4325X250N, F.Cu at (-50.8, -24.3)
- added D15: ES1D, ES1D:DIOM4325X250N, F.Cu at (-52.0, -15.9)
- added D16: LED, LED_SMD:LED_0603_1608Metric_Pad1.05x0.95mm_HandSolder, F.Cu at (-82.7, 10.4)
- added D4: ES1D, ES1D:DIOM4325X250N, F.Cu at (-50.8, -49.0)
- added D5: ES1D, ES1D:DIOM4325X250N, F.Cu at (-50.8, -44.9)
- added D6: ES1D, ES1D:DIOM4325X250N, F.Cu at (-50.8, -40.8)
- added D9: ES1D, ES1D:DIOM4325X250N, F.Cu at (-50.8, -36.7)
- added FB1: BLM18AG601SN1D, BLM18AG601SN1D:BEADC1608X95N, F.Cu at (-82.9, 12.9)
- added INT1: 01x04, Connector_JST:JST_PH_B4B-PH-K_1x04_P2.00mm_Vertical, F.Cu at (19.3, 55.2)
- added L1: 33uH, Inductor_SMD:L_Bourns_SRR1260, F.Cu at (-111.6, 21.7)
- added L2: 68uH, Inductor_SMD:L_Bourns_SRR1260, F.Cu at (-111.6, 35.8)
- added L3: 82683C, 82683C:FUSE_MF-USMFLAB, F.Cu at (-76.6, 49.9)
- added L4: 82103C, 82103C:IND_8200_MUR, F.Cu at (-71.4, 12.1)
- added PGND1: Conn_01x01, Connector_Wire:SolderWire-2.5sqmm_1x01_D2.4mm_OD3.6mm, F.Cu at (55.0, 54.0)
- added PH1: 01x03, Connector_Wire:SolderWire-2.5sqmm_1x03_P7.2mm_D2.4mm_OD3.6mm, F.Cu at (73.7, 37.0)
- added PRO1: 01x06, Connector_JST:JST_PH_B6B-PH-K_1x06_P2.00mm_Vertical, F.Cu at (5.50, 46.0)
- added PVCC1: Conn_01x01, Connector_Wire:SolderWire-2.5sqmm_1x01_D2.4mm_OD3.6mm, F.Cu at (55.0, 6.00)
- added Q1: SUD90330E, sud90330e:TO-252-2, F.Cu at (62.5, 15.0)
- added Q2: SUD90330E, sud90330e:TO-252-2, F.Cu at (51.0, 15.0)
- added Q3: SUD90330E, sud90330e:TO-252-2, F.Cu at (62.5, 30.0)
- added Q4: SUD90330E, sud90330e:TO-252-2, F.Cu at (51.0, 30.0)
- added Q5: SUD90330E, sud90330e:TO-252-2, F.Cu at (62.5, 45.0)
- added Q6: SUD90330E, sud90330e:TO-252-2, F.Cu at (51.0, 45.0)
- added R1: 5, Resistor_SMD:R_0603_1608Metric, F.Cu at (-32.4, 24.4)
- added R10: 4.7k, Resistor_SMD:R_0603_1608Metric, F.Cu at (-24.4, 16.8)
- added R11: 120, Resistor_SMD:R_0603_1608Metric, F.Cu at (-98.5, 36.8)
- added R12: 10, Resistor_SMD:R_0603_1608Metric, F.Cu at (-98.5, 39.3)
- added R13: 10, Resistor_SMD:R_0603_1608Metric, F.Cu at (-98.5, 41.8)
- added R14: 220, Resistor_SMD:R_0603_1608Metric, F.Cu at (-98.5, 44.3)
- added R15: 220, Resistor_SMD:R_0603_1608Metric, F.Cu at (-94.5, 31.8)
- added R16: 10K, Resistor_SMD:R_0603_1608Metric, F.Cu at (-94.5, 34.3)
- added R17: 10K, Resistor_SMD:R_0603_1608Metric, F.Cu at (-94.5, 36.8)
- added R18: 220, Resistor_SMD:R_0603_1608Metric, F.Cu at (-94.5, 39.3)
- added R19: 5mOhm, Resistor_SMD:R_2512_6332Metric, B.Cu at (65.0, 30.0)
- added R2: 47, Resistor_SMD:R_1206_3216Metric, F.Cu at (41.0, 12.9)
- added R20: 5mOhm, Resistor_SMD:R_2512_6332Metric, B.Cu at (65.0, 22.8)
- added R21: 5mOhm, Resistor_SMD:R_2512_6332Metric, B.Cu at (65.0, 37.2)
- added R3: 47, Resistor_SMD:R_1206_3216Metric, F.Cu at (39.0, 20.0)
- added R4: 5, Resistor_SMD:R_0603_1608Metric, F.Cu at (-28.4, 16.8)
- added R5: 47, Resistor_SMD:R_1206_3216Metric, F.Cu at (41.0, 27.9)
- added R6: 47, Resistor_SMD:R_1206_3216Metric, F.Cu at (39.0, 35.0)
- added R7: 5, Resistor_SMD:R_0603_1608Metric, F.Cu at (-28.4, 24.4)
- added R8: 47, Resistor_SMD:R_1206_3216Metric, F.Cu at (41.0, 42.9)
- added R9: 47, Resistor_SMD:R_1206_3216Metric, F.Cu at (39.0, 50.0)
- added STEP1: 01x02, Connector_JST:JST_PH_B2B-PH-K_1x02_P2.00mm_Vertical, F.Cu at (5.50, 27.3)
- added SW1: SW_Push, Button_Switch_SMD:SW_Push_1P1T_NO_CK_KMR2, F.Cu at (-76.0, 40.8)
- added SW2: SW_Push, Button_Switch_SMD:SW_Push_1P1T_NO_CK_KMR2, F.Cu at (-76.0, 45.5)
- added U1: IRS2104, Package_SO:SOIC-8_3.9x4.9mm_P1.27mm, F.Cu at (35.0, 15.0)
- added U12: AMC1311, AMC1311DWVR:DWV0008A, B.Cu at (29.0, 45.0)
- added U13: AMC1311, AMC1311DWVR:DWV0008A, B.Cu at (29.0, 15.0)
- added U14: CME0512S3C, CME0512S3C:CME_SC_MUR, F.Cu at (25.2, 56.0)
- added U15: CME0303S3C, CME0512S3C:CME_SC_MUR, F.Cu at (25.2, 7.50)
- added U16: INA241A2xD, Package_SO:SOIC-8_3.9x4.9mm_P1.27mm, B.Cu at (64.8, 44.5)
- added U2: IRS2104, Package_SO:SOIC-8_3.9x4.9mm_P1.27mm, F.Cu at (35.0, 30.0)
- added U3: IRS2104, Package_SO:SOIC-8_3.9x4.9mm_P1.27mm, F.Cu at (35.0, 45.0)
- added U4: ISO7740DWR, ISO7740DWR:SOIC127P1030X265-16N, B.Cu at (29.0, 30.0)
- added VCC1: 01x02, Connector_Wire:SolderWire-0.5sqmm_1x02_P4.6mm_D0.9mm_OD2.1mm, F.Cu at (13.9, 7.40)
- added Y1: ECS-80-20-18-TR, ECS-80-18-23B-JTN-TR:XTAL_ECS-80-20-18-TR, F.Cu at (-93.2, 0.38)
- D17, D18: footprint Diode_THT:D_DO-201AD_P15.24mm_Horizontal -> Diode_SMD:D_SMC
- U10: value INA241A3xD -> REF3020; footprint Package_SO:SOIC-8_3.9x4.9mm_P1.27mm -> Package_TO_SOT_SMD:SOT-23
- U11: value INA241A3xD -> INA241A2xD; moved to B.Cu
- U7: footprint Package_TO_SOT_THT:TO-220-3_Vertical -> Package_TO_SOT_SMD:SOT-223
- moved U9 302.2 mm to (-137.4, 3.20)
- moved U8 272.5 mm to (-107.9, -3.83)
- moved U6 264.8 mm to (-71.0, -6.64)
- moved U7 186.9 mm to (-74.4, 34.4)
- moved U10 180.7 mm to (-62.3, 61.5)
- moved D17 169.5 mm to (-73.9, 18.6)
- moved D18 165.2 mm to (-73.9, 26.3)
- moved U5 159.4 mm to (17.1, 39.9)
- moved U11 88.1 mm to (64.8, 15.1), turned to 180 degrees
Connections:
- U10 pad 1: B_IN- -> +3.3VIS
- U10 pad 2: PGND -> CS_REF
- U11 pad 7: +12VIS -> CS_REF
Routing:
- net PGND: track 0.00 -> 53.2 mm
- net PVCC: track 0.00 -> 46.7 mm
- net PB_CS: track 0.00 -> 27.0 mm, vias 0 -> 1
- net A_IN+: track 0.00 -> 15.8 mm, vias 0 -> 1
- net C_IN+: track 0.00 -> 14.5 mm, vias 0 -> 1
- net Net-(U2-VS): track 0.00 -> 7.83 mm
- net Net-(U3-VS): track 0.00 -> 7.71 mm
- net Net-(U1-VS): track 0.00 -> 7.22 mm
- net A_IN-: track 0.00 -> 6.14 mm
- net PB: track 0.00 -> 6.08 mm
- net C_IN-: track 0.00 -> 5.94 mm
- net Net-(U3-HO): track 0.00 -> 4.03 mm
- net Net-(U1-HO): track 0.00 -> 4.03 mm
- net Net-(U2-HO): track 0.00 -> 4.03 mm
- net Net-(D1-K): track 0.00 -> 3.94 mm
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- added copper zone on B.Cu, net PGND
Other:
- board outline added: 80 x 60 mm
- copper layers 2 -> 4
- board text added: "PA"
- board text added: "PB"
- board text added: "PC"
