File: 03_boards/00_bridge_driver/03_kicad/01_main/main.kicad_sch (KiCad schematic)
At the start: 48 parts, among them J1 01x02, SW1 SW_Push, SW2 SW_Push, U14 CME0512S3C, U15 CME0303S3C, U5 STM32G431K8Tx, U6 MAX3485, U7 LD1117V33, U8 LM2596S-5, U9 LM2596S-12, Y1 ECS-80-20-18-TR

Commit message: Made it clear the values and updated the schematics.
Other:
- note added: "Isolated 3.3V Supply"
Changed lines of the file:
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@@
 		)
 	)
-	(text "Isolated 12V Supply"
+	(text "Isolated 3.3V Supply"
 		(exclude_from_sim no)
-		(at 60.198 134.366 0)
+		(at 60.706 134.366 0)
 		(effects
 			(font

Commit message: Initial PCB modelling work
Parts:
- added J2, J3: Conn_01x01, Connector_Wire:SolderWire-2.5sqmm_1x01_D2.4mm_OD3.6mm, symbol Connector_Generic:Conn_01x01
- J1: footprint Connector_Wire:SolderWire-1sqmm_1x02_P7.8mm_D1.4mm_OD3.9mm -> Connector_Wire:SolderWire-0.5sqmm_1x02_P4.6mm_D0.9mm_OD2.1mm
Connections:
- net PGND: now also J3.1 (Pin_1)
- new net PVCC: J2.1 (Pin_1)
Other:
- note added: "Power-Side"
- note added: "WARNING: For current sensing, use either the `1 mΩ`, `5 mΩ`, or `10 mΩ` shunt resistor depending on your expected current."
- note removed: "WARNING: For current sensing, use either the `1 mΩ`, `3 mΩ`, or `10 mΩ` shunt resistor. Do not use more than a single path, or the driver will not function correctly."
- moved on the sheet: CAN1, INT1, J1, PH1, PRO1, STEP1

Commit message: Added work so far on bridge driver. Took some pics and updates readmes.
Parts:
- PH1: footprint Connector_Wire:SolderWire-2.5sqmm_1x03_P7.2mm_D2.4mm_OD3.6mm_Relief -> Connector_Wire:SolderWire-2.5sqmm_1x03_P7.2mm_D2.4mm_OD3.6mm
- renumbered J3 to PGND1, J2 to PVCC1, J1 to VCC1
Other:
- moved on the sheet: C12, C13, C14, C15, C16, C17, C18, C19, C20, C21, C22, C23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
