File: 03_boards/03_teensy_SFOC/03_kicad/01_main/teensy_SFOC/teensy_SFOC.kicad_sch (KiCad schematic)
At the start: 19 parts, among them U1 Teensy4.1, U2 MAX3485, U3 LD1117V33

Commit message: TeensySFOC & Armature REV 1
Parts:
- removed A1: SimpleFOC_Shield, PCM_arduino-library:Arduino_Uno_R2_Shield, symbol arduino-library:Arduino_Uno_R2_Shield
- added SFOC1: SimpleFOC Sheild, Module:Arduino_UNO_R3, symbol MCU_Module:Arduino_UNO_R3
- C1, C2, C3, C4: footprint Connector:FanPinHeader_1x04_P2.54mm_Vertical -> Capacitor_SMD:C_1206_3216Metric
- D1, D2: value DS -> 1N4148; footprint (none) -> Diode_SMD:D_SOD-123
- ENC1: footprint (none) -> Connector_JST:JST_XH_B5B-XH-A_1x05_P2.50mm_Vertical
- INT1: footprint (none) -> Connector_JST:JST_XH_B4B-XH-A_1x04_P2.50mm_Vertical
- PW1, SD1: footprint (none) -> Connector_JST:JST_XH_B2B-XH-A_1x02_P2.50mm_Vertical
- R1, R2, R3, R4, R5: footprint (none) -> Resistor_SMD:R_1206_3216Metric
- U1: footprint (none) -> teensy_library:Teensy41
- U3: footprint Package_TO_SOT_THT:TO-220-3_Vertical -> Package_TO_SOT_SMD:SOT-223-3_TabPin2
Connections:
- net CS1: now also U1.36 (14_A0_TX3_SPDIF_OUT); no longer D2.2 (A), R5.2
- net DIR: now also U1.14 (12_MISO_MQSL)
- net GND: now also SFOC1.29 (GND), SFOC1.6 (GND), SFOC1.7 (GND)
- net IN1: now also U1.7 (5_IN2), SFOC1.20 (D5)
- net IN2: now also U1.8 (6_OUT1D), SFOC1.24 (D9)
- net IN3: now also U1.9 (7_RX2_OUT1A), SFOC1.21 (D6)
- net INC_A: now also U1.11 (9_OUT1C)
- net INC_B: now also U1.10 (8_TX2_IN1)
- net INC_INDEX: now also U1.12 (10_CS_MQSR)
- net RC_RS: now also U1.2 (0_RX1_CRX2_CS1)
- net RS_DRI: now also U1.3 (1_TX1_CTX2_MISO1)
- net RS_EN: now also U1.4 (2_OUT2)
- net RS_TOG: now also U1.5 (3_LRCLK2)
- net SD: now also U1.6 (4_BCLK2), SFOC1.23 (D8)
- net SF_CS1: now also SFOC1.9 (A0)
- net SF_CS2: now also R5.2, SFOC1.11 (A2); no longer R5.1
- net STEP: now also U1.13 (11_MOSI_CTX1)
- net CS2: now reaches U1.37 (15_A1_RX3_SPDIF_IN)
- net CS2: now also D2.2 (A), R5.1
- no-connect marks 28 -> 68
Other:
- note added: "SimpleFOC Interface (Arduino Uno Shield)"
- note removed: "SimpleFOC Interface"
- moved on the sheet: R5
