File: 03_boards/01_armature_board/03_kicad/01_main/main.kicad_pcb (KiCad board)
At the start: 2 copper layers, 60 x 40 mm, 59 parts, among them U1 STM32G431K8Tx, U2 LD1117S33, U3 MAX3485, U4 ADXL343, U5 74HC4051, Y1 ECS-80-20-18-TR

Commit message: Week 0xB | TeensySFOC & began work on hybrid model. (#44)
* Initial work on TeensySFOC board

* Added SFOC readme

* Schematic and referencing in the readme

* TeensySFOC & Armature REV 1

* Updated readme

* Few changes.

* Updated sub-readme

* Breakout not integration

* Added note.

* Update README.md

* Update README.md

* Deleted concenptual design

* Removed old driver pcb images from readme

* Update README.md

* Initial work on hybird model.

* Added a citation at the bottom of the repo

* Updated common point readme

* Fixed formatting

* Removed old implementation images & BOM

* Removed space.

* Moved link downwards

* Changed status.

* Updating formatting

* Formatting fix

* Removed images of board

* Update readme.md

* Renaming files & fixing formatting

* Updating hybrid model stuff

* Fixing formatting

* Formatting updates.

* Fixing formatting
Parts:
- ENC1: footprint Connector_JST:JST_PH_B5B-PH-K_1x05_P2.00mm_Vertical -> Connector_JST:JST_XH_B5B-XH-A_1x05_P2.50mm_Vertical
- INT1: footprint Connector_JST:JST_PH_B4B-PH-K_1x04_P2.00mm_Vertical -> Connector_JST:JST_XH_B4B-XH-A_1x04_P2.50mm_Vertical
- moved RESET1 2.50 mm to (41.5, 36.0)
- moved INT1 1.00 mm to (11.5, 35.5)
- moved U3 0.74 mm to (12.5, 23.8)
- moved R3 0.74 mm to (13.3, 31.8)
- moved R1 0.50 mm to (12.0, 29.5)
- moved ENC1 0.50 mm to (25.0, 35.5)
- moved R2 0.49 mm to (14.1, 29.5)
Connections:
- U1 pad 26: unconnected-(U1-PB3-Pad26) -> SWO
- U1 pad 8: SWO -> unconnected-(U1-PA3-Pad8)
Routing:
- net GND: track 43.3 -> 47.7 mm
- net Net-(R17-Pad1): track 6.02 -> 7.47 mm
- net INC_Index: track 14.4 -> 15.3 mm
- net D_P: track 5.66 -> 6.45 mm
- net Net-(U3-B): track 2.61 -> 3.37 mm
- net INC_A: track 14.2 -> 14.9 mm
Other:
- board text added: "Armature Board REV 1"
- board text added: "Wgbowley 26-09-17"
- board text removed: "Armature Board REV 0"
- board text removed: "Wgbowley 26-08-01"
