File: 03_boards/01_armature_board/03_kicad/01_main/main.kicad_sch (KiCad schematic)
At the start: 58 parts, among them J1 01x04, J10 01x02, J11 01x02, J2 01x06, J3 01x05, J4 01x02, J5 01x02, J6 01x02, J7 01x02, J8 01x02, J9 01x02, SW1 SW_Push, SW2 SW_Push, U1 STM32G431K8Tx, U2 LD1117S33, U3 MAX3485, U4 ADXL343, U5 74HC4051, Y1 ECS-80-20-18-TR

Commit message: Schematic validation done moving to documentation before pcb
Parts:
- removed C24: 100nf, symbol Device:C_Small
- removed R4: 0Ω, symbol Device:R_Small
- added FB1: BLM18AG601SN1D, symbol Device:FerriteBead
- added R16, R17: 220, symbol Device:R
- C16, C17, C18, C19, C20, C21, C22, C23: value 100nf -> 10nf
Connections:
- net +3.3V: now also J10.2 (Pin_2), J11.2 (Pin_2), J4.2 (Pin_2), J5.2 (Pin_2), J6.2 (Pin_2), J7.2 (Pin_2), J8.2 (Pin_2), J9.2 (Pin_2), FB1.1, R16.2; no longer SW1.1, SW2.1
- net GND: now also SW2.2
- net NRST: now also R17.2; no longer SW2.2
- net TA1: now also C16.1, J4.1 (Pin_1), R8.2; no longer J4.2 (Pin_2)
- net TA2: now also C18.1, J6.1 (Pin_1), R10.2; no longer J6.2 (Pin_2)
- net TA3: now also C20.1, J8.1 (Pin_1), R12.2; no longer J8.2 (Pin_2)
- net TA4: now also C17.1, J5.1 (Pin_1), R9.2; no longer J5.2 (Pin_2)
- net TA5: now also C19.1, J7.1 (Pin_1), R11.2; no longer J7.2 (Pin_2)
- net TA6: now also C21.1, J9.1 (Pin_1), R13.2; no longer J9.2 (Pin_2)
- net TA7: now also C22.1, J10.1 (Pin_1), R14.2; no longer J10.2 (Pin_2)
- net TA8: now also C23.1, J11.1 (Pin_1), R15.2; no longer J11.2 (Pin_2)
- net VDDA: now also FB1.2
- new net: R16.1, SW1.1
- new net: R17.1, SW2.1
- no-connect marks 6 -> 7
Other:
- note added: "TA1-TA3"
- note added: "TA4-TA6"
- note added: "TA7-TA8"
- moved on the sheet: C13, C14, C15, C16, C17, C18, C19, C20, C21, C22, C23, C5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

Commit message: Validation finished & initial pre-pcb documentation done
Parts:
- added R18, R19: 0Ω, symbol Device:R_Small
Connections:
- net RS_DRI: now also R18.2
- net RS_RC: no longer U1.30 (PB7)
- net RS_TOG: now also U1.30 (PB7), R19.2
- net dn renamed RX
- net RX: now also R19.1
- net dp renamed TX
- net TX: now also R18.1
Other:
- note added: "RS Bypass (TX, RX)"
- moved on the sheet: C22

Commit message: Updated armature board footprints
Parts:
- C1, C10, C11, C12, C13, C14, C15, C16, C17, C18, C19, C20, C21, C22, C23, C3, C5, C6, C9: footprint (none) -> Capacitor_SMD:C_0603_1608Metric
- C4, C7, C8: footprint (none) -> Capacitor_SMD:C_1206_3216Metric
- D1: footprint (none) -> LED_SMD:LED_1206_3216Metric
- FB1: footprint (none) -> BLM18AG601SN1D:BEADC1608X95N
- J1: footprint (none) -> Connector_JST:JST_PH_B4B-PH-K_1x04_P2.00mm_Vertical
- J10, J11, J4, J5, J6, J7, J8, J9: footprint (none) -> Connector_JST:JST_PH_B2B-PH-K_1x02_P2.00mm_Vertical
- J2: footprint (none) -> Connector_JST:JST_PH_B6B-PH-K_1x06_P2.00mm_Vertical
- J3: footprint (none) -> Connector_JST:JST_PH_B5B-PH-K_1x05_P2.00mm_Vertical
- R1, R10, R11, R12, R13, R14, R15, R16, R17, R18, R19, R2, R3, R5, R6, R7, R8, R9: footprint (none) -> Resistor_SMD:R_0603_1608Metric
- SW1, SW2: footprint (none) -> Button_Switch_THT:SW_PUSH_6mm
- U5: footprint (none) -> 74HC4051:SSOP-16
- Y1: footprint ECS-80-20-18-TR:XTAL_ECS-80-20-18-TR -> ECS-80-18-23B-JTN-TR:XTAL_ECS-80-20-18-TR
Changed lines of the file:
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@@
 			)
 		)
-		(property "Footprint" ""
+		(property "Footprint" "Capacitor_SMD:C_1206_3216Metric"
 			(at 105.41 60.96 0)
 			(hide yes)
@@
 			)
 		)
-		(property "Footprint" ""
+		(property "Footprint" "Resistor_SMD:R_0603_1608Metric"
 			(at 61.468 137.16 90)
 			(hide yes)
@@
 			)
 		)
-		(property "Footprint" ""
+		(property "Footprint" "Connector_JST:JST_PH_B2B-PH-K_1x02_P2.00mm_Vertical"
 			(at 52.07 177.8 0)
 			(hide yes)
@@
 			)
 		)
-		(property "Footprint" ""
+		(property "Footprint" "Connector_JST:JST_PH_B2B-PH-K_1x02_P2.00mm_Vertical"
 			(at 82.55 132.08 0)
 			(hide yes)
@@
 			)
 		)
-		(property "Footprint" ""
+		(property "Footprint" "Connector_JST:JST_PH_B4B-PH-K_1x04_P2.00mm_Vertical"
 			(at 22.86 33.02 0)
 			(hide yes)
@@
 			)
 		)
-		(property "Footprint" ""
+		(property "Footprint" "Capacitor_SMD:C_0603_1608Metric"
 			(at 38.1 181.61 0)
 			(hide yes)
@@
 			)
 		)
-		(property "Footprint" ""
+		(property "Footprint" "Resistor_SMD:R_0603_1608Metric"
 			(at 250.952 71.12 90)
 			(hide yes)
@@
 			)
 		)
-		(property "Footprint" ""
+		(property "Footprint" "Resistor_SMD:R_0603_1608Metric"
 			(at 198.12 103.632 90)
 			(hide yes)
@@
 			)
 		)
-		(property "Footprint" ""
+		(property "Footprint" "74HC4051:SSOP-16"
 			(at 132.08 154.94 0)
 			(hide yes)
@@
 			)
 		)
-		(property "Footprint" "ECS-80-20-18-TR:XTAL_ECS-80-20-18-TR"
+		(property "Footprint" "ECS-80-18-23B-JTN-TR:XTAL_ECS-80-20-18-TR"
 			(at 161.29 78.74 0)
 			(hide yes)
@@
 			)
 		)
-		(property "Footprint" ""
+		(property "Footprint" "Connector_JST:JST_PH_B2B-PH-K_1x02_P2.00mm_Vertical"
 			(at 20.32 132.08 0)
 			(hide yes)
@@
 			)
 		)
-		(property "Footprint" ""
+		(property "Footprint" "Capacitor_SMD:C_0603_1608Metric"
 			(at 242.57 30.48 0)
 			(hide yes)
@@
 			)
 		)
-		(property "Footprint" ""
+		(property "Footprint" "Button_Switch_THT:SW_PUSH_6mm"
 			(at 250.19 100.33 0)
 			(hide yes)
@@
 			)
 		)
-		(property "Footprint" ""
+		(property "Footprint" "Resistor_SMD:R_0603_1608Metric"
 			(at 203.962 69.85 90)
 			(hide yes)
@@
 			)
 		)
-		(property "Footprint" ""
+		(property "Footprint" "Resistor_SMD:R_0603_1608Metric"
 			(at 61.468 182.88 90)
 			(hide yes)
@@
 			)
 		)
-		(property "Footprint" ""
+		(property "Footprint" "Button_Switch_THT:SW_PUSH_6mm"
 			(at 210.82 100.33 0)
 			(hide yes)
@@
 			)
 		)
-		(property "Footprint" ""
+		(property "Footprint" "Resistor_SMD:R_0603_1608Metric"
 			(at 29.718 160.02 90)
 			(hide yes)
@@
 			)
 		)
-		(property "Footprint" ""
+		(property "Footprint" "Connector_JST:JST_PH_B2B-PH-K_1x02_P2.00mm_Vertical"
 			(at 52.07 154.94 0)
 			(hide yes)
@@
 			)
 		)
-		(property "Footprint" ""
+		(property "Footprint" "Capacitor_SMD:C_0603_1608Metric"
 			(at 96.52 60.96 0)
 			(hide yes)
@@
 			)
 		)
-		(property "Footprint" ""
+		(property "Footprint" "Capacitor_SMD:C_0603_1608Metric"
 			(at 72.39 83.82 0)
 			(hide yes)
@@
 			)
 		)
-		(property "Footprint" ""
+		(property "Footprint" "LED_SMD:LED_1206_3216Metric"
 			(at 252.73 80.01 0)
 			(hide yes)
@@
 			)
 		)
-		(property "Footprint" ""
+		(property "Footprint" "Capacitor_SMD:C_0603_1608Metric"
 			(at 36.83 137.16 0)
 			(hide yes)
@@
 			)
 		)
-		(property "Footprint" ""
+		(property "Footprint" "Connector_JST:JST_PH_B2B-PH-K_1x02_P2.00mm_Vertical"
 			(at 20.32 154.94 0)
 			(hide yes)
@@
 			)
 		)
-		(property "Footprint" ""
+		(property "Footprint" "Capacitor_SMD:C_0603_1608Metric"
 			(at 68.58 137.16 0)
 			(hide yes)
@@
 			)
 		)
-		(property "Footprint" ""
+		(property "Footprint" "Resistor_SMD:R_0603_1608Metric"
 			(at 158.75 102.87 0)
 			(hide yes)
@@
 			)
 		)
-		(property "Footprint" ""
+		(property "Footprint" "Connector_JST:JST_PH_B2B-PH-K_1x02_P2.00mm_Vertical"
 			(at 21.59 177.8 0)
 			(hide yes)
@@
 			)
 		)
-		(property "Footprint" ""
+		(property "Footprint" "Capacitor_SMD:C_0603_1608Metric"
 			(at 152.4 82.55 0)
 			(hide yes)
@@
 			)
 		)
-		(property "Footprint" ""
+		(property "Footprint" "Resistor_SMD:R_0603_1608Metric"
 			(at 203.962 30.48 90)
 			(hide yes)
@@
 			)
 		)
-		(property "Footprint" ""
+		(property "Footprint" "Capacitor_SMD:C_0603_1608Metric"
 			(at 66.04 34.29 0)
 			(hide yes)
@@
 			)
 		)
-		(property "Footprint" ""
+		(property "Footprint" "Resistor_SMD:R_0603_1608Metric"
 			(at 240.03 103.632 90)
 			(hide yes)
@@
 			)
 		)
-		(property "Footprint" ""
+		(property "Footprint" "Capacitor_SMD:C_0603_1608Metric"
 			(at 254 30.48 0)
 			(hide yes)
@@
 			)
 		)
-		(property "Footprint" ""
+		(property "Footprint" "Capacitor_SMD:C_0603_1608Metric"
 			(at 49.53 31.75 0)
 			(hide yes)
@@
 			)
 		)
-		(property "Footprint" ""
+		(property "Footprint" "Resistor_SMD:R_0603_1608Metric"
 			(at 61.468 160.02 90)
 			(hide yes)
@@
 			)
 		)
-		(property "Footprint" ""
+		(property "Footprint" "Resistor_SMD:R_0603_1608Metric"
 			(at 127 29.718 90)
 			(hide yes)
@@
 			)
 		)
-		(property "Footprint" ""
+		(property "Footprint" "Connector_JST:JST_PH_B2B-PH-K_1x02_P2.00mm_Vertical"
 			(at 82.55 154.94 0)
 			(hide yes)
@@
 			)
 		)
-		(property "Footprint" ""
+		(property "Footprint" "Capacitor_SMD:C_0603_1608Metric"
 			(at 168.91 82.55 0)
 			(hide yes)
@@
 			)
 		)
-		(property "Footprint" ""
+		(property "Footprint" "Capacitor_SMD:C_0603_1608Metric"
 			(at 99.06 137.16 0)
 			(hide yes)
@@
 			)
 		)
-		(property "Footprint" ""
+		(property "Footprint" "Capacitor_SMD:C_0603_1608Metric"
 			(at 68.58 160.02 0)
 			(hide yes)
@@
 			)
 		)
-		(property "Footprint" ""
+		(property "Footprint" "Resistor_SMD:R_0603_1608Metric"
 			(at 127 39.878 90)
 			(hide yes)
@@
 			)
 		)
-		(property "Footprint" ""
+		(property "Footprint" "Connector_JST:JST_PH_B2B-PH-K_1x02_P2.00mm_Vertical"
 			(at 52.07 132.08 0)
 			(hide yes)
@@
 			)
 		)
-		(property "Footprint" ""
+		(property "Footprint" "Capacitor_SMD:C_0603_1608Metric"
 			(at 231.14 110.49 0)
 			(hide yes)
@@
 			)
 		)
-		(property "Footprint" ""
+		(property "Footprint" "Resistor_SMD:R_0603_1608Metric"
 			(at 91.948 160.02 90)
 			(hide yes)
@@
 			)
 		)
-		(property "Footprint" ""
+		(property "Footprint" "Capacitor_SMD:C_1206_3216Metric"
 			(at 91.44 34.29 0)
 			(hide yes)
@@
 			)
 		)
-		(property "Footprint" ""
+		(property "Footprint" "BLM18AG601SN1D:BEADC1608X95N"
 			(at 77.47 57.658 90)
 			(hide yes)
@@
 			)
 		)
-		(property "Footprint" ""
+		(property "Footprint" "Resistor_SMD:R_0603_1608Metric"
 			(at 30.988 182.88 90)
 			(hide yes)
@@
 			)
 		)
-		(property "Footprint" ""
+		(property "Footprint" "Capacitor_SMD:C_0603_1608Metric"
 			(at 85.09 60.96 0)
 			(hide yes)
@@
 			)
 		)
-		(property "Footprint" ""
+		(property "Footprint" "Connector_JST:JST_PH_B5B-PH-K_1x05_P2.00mm_Vertical"
 			(at 22.86 95.25 0)
 			(hide yes)
@@
 			)
 		)
-		(property "Footprint" ""
+		(property "Footprint" "Connector_JST:JST_PH_B6B-PH-K_1x06_P2.00mm_Vertical"
 			(at 22.86 59.69 0)
 			(hide yes)
@@
 			)
 		)
-		(property "Footprint" ""
+		(property "Footprint" "Resistor_SMD:R_0603_1608Metric"
 			(at 29.718 137.16 90)
 			(hide yes)
@@
 			)
 		)
-		(property "Footprint" ""
+		(property "Footprint" "Capacitor_SMD:C_0603_1608Metric"
 			(at 68.58 182.88 0)
 			(hide yes)
@@
 			)
 		)
-		(property "Footprint" ""
+		(property "Footprint" "Resistor_SMD:R_0603_1608Metric"
 			(at 91.948 137.16 90)
 			(hide yes)
@@
 			)
 		)
-		(property "Footprint" ""
+		(property "Footprint" "Resistor_SMD:R_0603_1608Metric"
 			(at 158.75 109.22 0)
 			(hide yes)
@@
 			)
 		)
-		(property "Footprint" ""
+		(property "Footprint" "Resistor_SMD:R_0603_1608Metric"
 			(at 121.158 33.02 90)
 			(hide yes)
@@
 			)
 		)
-		(property "Footprint" ""
+		(property "Footprint" "Capacitor_SMD:C_0603_1608Metric"
 			(at 99.06 160.02 0)
 			(hide yes)
@@
 			)
 		)
-		(property "Footprint" ""
+		(property "Footprint" "Capacitor_SMD:C_0603_1608Metric"
 			(at 36.83 158.75 0)
 			(hide yes)
@@
 			)
 		)
-		(property "Footprint" ""
+		(property "Footprint" "Capacitor_SMD:C_1206_3216Metric"
 			(at 115.57 60.96 0)
 			(hide yes)
@@
 			)
 		)
-		(property "Footprint" ""
+		(property "Footprint" "Capacitor_SMD:C_0603_1608Metric"
 			(at 219.71 110.49 0)
 			(hide yes)

Commit message: Saving pcb layout work for armature board
Parts:
- PRO1: renamed from J2; footprint Connector_JST:JST_PH_B6B-PH-K_1x06_P2.00mm_Vertical -> Connector_PinHeader_2.54mm:PinHeader_2x03_P2.54mm_Vertical
- SW1, SW2: footprint Button_Switch_THT:SW_PUSH_6mm -> Button_Switch_SMD:SW_Push_1P1T_NO_CK_KMR2
- renumbered J3 to ENC1, J1 to INT1, J4 to NTC1, J5 to NTC2, J10 to NTC3, J6 to NTC4, J7 to NTC5, J11 to NTC6, J8 to NTC7, J9 to NTC8
Connections:
- net TA2: now also C17.1, NTC2.1 (Pin_1), R9.2; no longer C18.1, NTC4.1 (Pin_1), R10.2
- net TA3: now also C22.1, NTC3.1 (Pin_1), R14.2; no longer C20.1, NTC7.1 (Pin_1), R12.2
- net TA4: now also C18.1, NTC4.1 (Pin_1), R10.2; no longer C17.1, NTC2.1 (Pin_1), R9.2
- net TA6: now also C23.1, NTC6.1 (Pin_1), R15.2; no longer C21.1, NTC8.1 (Pin_1), R13.2
- net TA7: now also C20.1, NTC7.1 (Pin_1), R12.2; no longer C22.1, NTC3.1 (Pin_1), R14.2
- net TA8: now also C21.1, NTC8.1 (Pin_1), R13.2; no longer C23.1, NTC6.1 (Pin_1), R15.2
Changed lines of the file:
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@@
 		)
 	)
-	(global_label "TA2"
+	(global_label "TA4"
 		(shape output)
 		(at 39.37 154.94 0)
@@
 		)
 	)
-	(global_label "TA6"
+	(global_label "TA8"
 		(shape output)
 		(at 71.12 177.8 0)
@@
 		)
 	)
-	(global_label "TA4"
+	(global_label "TA2"
 		(shape output)
 		(at 71.12 132.08 0)
@@
 		)
 	)
-	(global_label "TA3"
+	(global_label "TA7"
 		(shape output)
 		(at 40.64 177.8 0)
@@
 		)
 	)
-	(global_label "TA7"
+	(global_label "TA3"
 		(shape output)
 		(at 101.6 132.08 0)
@@
 		)
 	)
-	(global_label "TA8"
+	(global_label "TA6"
 		(shape output)
 		(at 101.6 154.94 0)
@@
 		(in_pos_files yes)
 		(dnp no)
-		(property "Reference" "J9"
-			(at 51.562 170.688 0)
+		(property "Reference" "NTC8"
+			(at 52.832 170.688 0)
 			(show_name no)
 			(do_not_autoplace no)
@@
 			(project "main"
 				(path "/d7317114-a4fd-40b5-9eea-fb013c7aed3d"
-					(reference "J9")
+					(reference "NTC8")
 					(unit 1)
 				)
@@
 		(in_pos_files yes)
 		(dnp no)
-		(property "Reference" "J10"
-			(at 82.55 124.968 0)
+		(property "Reference" "NTC3"
+			(at 83.312 124.968 0)
 			(show_name no)
 			(do_not_autoplace no)
@@
 			(project "main"
 				(path "/d7317114-a4fd-40b5-9eea-fb013c7aed3d"
-					(reference "J10")
+					(reference "NTC3")
 					(unit 1)
 				)
@@
 		(in_pos_files yes)
 		(dnp no)
-		(property "Reference" "J1"
-			(at 22.86 22.606 0)
+		(property "Reference" "INT1"
+			(at 22.86 23.368 0)
 			(show_name no)
 			(do_not_autoplace no)
@@
 		)
 		(property "Value" "01x04"
-			(at 22.86 24.638 0)
+			(at 24.13 25.146 0)
 			(show_name no)
 			(do_not_autoplace no)
@@
 			(project "main"
 				(path "/d7317114-a4fd-40b5-9eea-fb013c7aed3d"
-					(reference "J1")
+					(reference "INT1")
 					(unit 1)
 				)
@@
 		(in_pos_files yes)
 		(dnp no)
-		(property "Reference" "J4"
-			(at 19.812 124.968 0)
+		(property "Reference" "NTC1"
+			(at 21.082 124.968 0)
 			(show_name no)
 			(do_not_autoplace no)
@@
 			(project "main"
 				(path "/d7317114-a4fd-40b5-9eea-fb013c7aed3d"
-					(reference "J4")
+					(reference "NTC1")
 					(unit 1)
 				)
@@
 			)
 		)
-		(property "Footprint" "Button_Switch_THT:SW_PUSH_6mm"
+		(property "Footprint" "Button_Switch_SMD:SW_Push_1P1T_NO_CK_KMR2"
 			(at 250.19 100.33 0)
 			(hide yes)
@@
 			)
 		)
-		(property "Footprint" "Button_Switch_THT:SW_PUSH_6mm"
+		(property "Footprint" "Button_Switch_SMD:SW_Push_1P1T_NO_CK_KMR2"
 			(at 210.82 100.33 0)
 			(hide yes)
@@
 		(in_pos_files yes)
 		(dnp no)
-		(property "Reference" "J7"
-			(at 51.562 147.828 0)
+		(property "Reference" "NTC5"
+			(at 52.832 147.828 0)
 			(show_name no)
 			(do_not_autoplace no)
@@
 			(project "main"
 				(path "/d7317114-a4fd-40b5-9eea-fb013c7aed3d"
-					(reference "J7")
+					(reference "NTC5")
 					(unit 1)
 				)
@@
 		(in_pos_files yes)
 		(dnp no)
-		(property "Reference" "J6"
-			(at 19.812 147.828 0)
+		(property "Reference" "NTC4"
+			(at 21.082 147.828 0)
 			(show_name no)
 			(do_not_autoplace no)
@@
 			(project "main"
 				(path "/d7317114-a4fd-40b5-9eea-fb013c7aed3d"
-					(reference "J6")
+					(reference "NTC4")
 					(unit 1)
 				)
@@
 		(in_pos_files yes)
 		(dnp no)
-		(property "Reference" "J8"
-			(at 21.082 170.688 0)
+		(property "Reference" "NTC7"
+			(at 22.352 170.688 0)
 			(show_name no)
 			(do_not_autoplace no)
@@
 			(project "main"
 				(path "/d7317114-a4fd-40b5-9eea-fb013c7aed3d"
-					(reference "J8")
+					(reference "NTC7")
 					(unit 1)
 				)
@@
 		(in_pos_files yes)
 		(dnp no)
-		(property "Reference" "J11"
-			(at 82.804 147.828 0)
+		(property "Reference" "NTC6"
+			(at 83.312 147.828 0)
 			(show_name no)
 			(do_not_autoplace no)
@@
 			(project "main"
 				(path "/d7317114-a4fd-40b5-9eea-fb013c7aed3d"
-					(reference "J11")
+					(reference "NTC6")
 					(unit 1)
 				)
@@
 		(in_pos_files yes)
 		(dnp no)
-		(property "Reference" "J5"
-			(at 51.562 124.968 0)
+		(property "Reference" "NTC2"
+			(at 52.832 124.968 0)
 			(show_name no)
 			(do_not_autoplace no)
@@
 			(project "main"
 				(path "/d7317114-a4fd-40b5-9eea-fb013c7aed3d"
-					(reference "J5")
+					(reference "NTC2")
 					(unit 1)
 				)
@@
 		(in_pos_files yes)
 		(dnp no)
-		(property "Reference" "J3"
-			(at 22.86 84.328 0)
+		(property "Reference" "ENC1"
+			(at 23.114 85.344 0)
 			(show_name no)
 			(do_not_autoplace no)
@@
 		)
 		(property "Value" "01x05"
-			(at 22.86 86.868 0)
+			(at 24.13 87.122 0)
 			(show_name no)
 			(do_not_autoplace no)
@@
 			(project "main"
 				(path "/d7317114-a4fd-40b5-9eea-fb013c7aed3d"
-					(reference "J3")
+					(reference "ENC1")
 					(unit 1)
 				)
@@
 		(in_pos_files yes)
 		(dnp no)
-		(property "Reference" "J2"
-			(at 22.86 46.736 0)
+		(property "Reference" "PRO1"
+			(at 24.13 47.498 0)
 			(show_name no)
 			(do_not_autoplace no)
@@
 		)
 		(property "Value" "01x06"
-			(at 22.86 48.514 0)
+			(at 24.384 49.276 0)
 			(show_name no)
 			(do_not_autoplace no)
@@
 			)
 		)
-		(property "Footprint" "Connector_JST:JST_PH_B6B-PH-K_1x06_P2.00mm_Vertical"
+		(property "Footprint" "Connector_PinHeader_2.54mm:PinHeader_2x03_P2.54mm_Vertical"
 			(at 22.86 59.69 0)
 			(hide yes)
@@
 			(project "main"
 				(path "/d7317114-a4fd-40b5-9eea-fb013c7aed3d"
-					(reference "J2")
+					(reference "PRO1")
 					(unit 1)
 				)
