File: 03_boards/00_armature_board/03_kicad/01_main/main.kicad_sch (KiCad schematic)
At the start: 59 parts, among them U1 STM32G431K8Tx, U2 LD1117S33, U3 MAX3485, U4 ADXL343, U5 74HC4051, Y1 ECS-80-20-18-TR

Commit message: Final magnetic search and updated schematic for armature board.
Parts:
- U1: value STM32G431K8Tx -> STM32G431
Changed lines of the file:
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@@
 			)
 		)
-		(property "Value" "STM32G431K8Tx"
+		(property "Value" "STM32G431"
 			(at 228.092 83.566 0)
 			(show_name no)
